File: QATCH openQCM PCB.kicad_pcb (KiCad board)
At the start: 2 copper layers, 60 x 82.2 mm, 79 parts, among them CN1 1727010, IC1 MIC5219-5.0YM5-TR, IC2 MAX31855KASA, J1 22057025, J2 20021111-00010T4LF, J3 0022152056, P1 PPTC241LFBN-RC, P2 PPTC241LFBN-RC, Q1 MMBT3904, Q2 MMBT3904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

Commit message: Committing local changes, adding cap bank and fix 5V pullups
Parts:
- added C27: 0.1uF, Footprints:CAP_KGM21_KAV, F.Cu at (140.6, 139.4)
- added C28: 0.1uF, Footprints:CAP_KGM21_KAV, F.Cu at (143.0, 139.4)
- added C29: 0.1uF, Footprints:CAP_KGM21_KAV, F.Cu at (145.4, 139.4)
- added C30: 0.1uF, Footprints:CAP_KGM21_KAV, F.Cu at (147.8, 139.4)
- added C31: 0.1uF, Footprints:CAP_KGM21_KAV, F.Cu at (150.2, 139.4)
- added R28: 1.5k, Footprints:BO_CR0805, F.Cu at (149.6, 90.4)
- added R29: 3k, Footprints:RC0805N_YAG, F.Cu at (149.7, 92.7)
- moved R8 24.3 mm to (134.6, 96.4), turned to 0 degrees
- moved R10 16.6 mm to (137.0, 101.0), turned to 90 degrees
- moved R1 9.95 mm to (142.9, 131.4)
- moved C22 7.85 mm to (137.3, 137.8)
- moved IC1 7.85 mm to (131.0, 137.9)
- moved R2 1.82 mm to (136.7, 113.8), turned to 180 degrees
- turned TP1 to -90 degrees
- turned TP2 to -90 degrees
- turned TP3 to -90 degrees
Connections:
- net /A0 renamed /14_A0(PWM)
- net /A14 renamed /33(PWM)
- net /A15(VREF) renamed /34(VREF)
- net /A16(PWM) renamed /35
- net /A17(PWM) renamed /36(PWM)
- net /A18 renamed /37(PWM)
- net /A19(GAIN) renamed /A14(GAIN)
- net /A20 renamed /39_A15
- net /D41 renamed /A17(SENSE)
- P2 pad 8: /A21 -> /A16(DETECT)
- R1 pad 2: +5V -> +3.3V
- R10 pad 2: +5V -> +3.3V
- R2 pad 2: +5V -> +3.3V
- R8 pad 2: +5V -> +3.3V
Routing:
- net +5V: track 264.6 -> 287.7 mm, vias 8 -> 10
- net /A16(DETECT): track 0.00 -> 10.5 mm
- net +3.3V: track 116.0 -> 126.1 mm, vias 1 -> 3
- net /Vin: track 91.2 -> 99.1 mm
- net /A8(W_CLK): track 27.9 -> 21.0 mm, vias 3 -> 2
- net /A5(SCL0): track 44.7 -> 46.4 mm
- net GND: vias 0 -> 4
- net (no net): vias 4 -> 0
