File: QATCH openQCM PCB.kicad_sch (KiCad schematic)
At the start: 79 parts, among them CN1 1727010, IC1 MIC5219-5.0YM5-TR, IC2 MAX31855KASA, J1 22057025, J2 20021111-00010T4LF, J3 0022152056, P1 PPTC241LFBN-RC, P2 PPTC241LFBN-RC, Q1 MMBT3904, Q2 MMBT3904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

Commit message: Committing local changes, adding cap bank and fix 5V pullups
Parts:
- added C27, C28, C29, C30, C31: 0.1uF, CAP_KGM21_KAV, symbol Symbols:KGM21NR71H104KT
- added R28: 1.5k, RC0805N_YAG, symbol Symbols:RC0805FR-071K5L
- added R29: 3k, RC0805N_YAG, symbol Symbols:RC0805FR-073KL
Connections:
- net +3.3V: now also R1.2, R10.2, R2.2, R8.2
- net +5V: now also R29.2; no longer R1.2, R10.2, R2.2, R8.2
- net GND: now also C27.2, C28.2, C29.2, C30.2, C31.2, R28.2
- net Vin: now also C27.1, C28.1, C29.1, C30.1, C31.1
- net A0 renamed 14_A0(PWM)
- net A14 renamed 33(PWM)
- net A15(VREF) renamed 34(VREF)
- net A16(PWM) renamed 35
- net A17(PWM) renamed 36(PWM)
- net A18 renamed 37(PWM)
- net A19(GAIN) renamed A14(GAIN)
- net A20 renamed 39_A15
- net A21 renamed A16(DETECT)
- net A16(DETECT): now also R28.1, R29.1
- net D41 renamed A17(SENSE)
- no-connect marks 22 -> 27
Other:
- note added: "Regulated Voltage Capacitor Bank"
- note added: "Source Voltage Capacitor Bank"
- note added: "Source Voltage Detector"
- note added: "Unused"
- note removed: "Capacitor Bank"
